File: kicadFiles/shark.sch (KiCad schematic (older format))
At the start: 262 parts, among them J1 USB_C_Receptacle, J2 Conn_01x04_Male, J3 Conn_01x04_Male, J4 Conn_01x04_Male, Q1 AO4406AL, SW1 MXSwitch, SW10 MXSwitch, SW11 MXSwitch, SW12 MXSwitch, SW13 MXSwitch, SW14 MXSwitch, SW15 MXSwitch, SW16 MXSwitch, SW17 MXSwitch, SW18 MXSwitch, SW19 MXSwitch, SW2 MXSwitch, SW20 MXSwitch, SW21 MXSwitch, SW22 MXSwitch, SW23 MXSwitch, SW24 MXSwitch, SW25 MXSwitch, SW26 MXSwitch, SW27 MXSwitch, SW28 MXSwitch, SW29 MXSwitch, SW3 MXSwitch, SW30 MXSwitch, SW31 MXSwitch, SW32 MXSwitch, SW33 MXSwitch, SW34 MXSwitch, SW35 MXSwitch, SW36 MXSwitch, SW37 MXSwitch, SW38 MXSwitch, SW39 MXSwitch, SW4 MXSwitch, SW40 MXSwitch, SW41 MXSwitch, SW42 MXSwitch, SW43 MXSwitch, SW44 MXSwitch, SW45 MXSwitch, SW46 MXSwitch, SW47 MXSwitch, SW48 MXSwitch, SW49 MXSwitch, SW5 MXSwitch, SW50 MXSwitch, SW51 MXSwitch, SW6 MXSwitch, SW7 MXSwitch, SW8 MXSwitch, SW9 MXSwitch, U1 STM32F303CCT6, U2 MCP1700-3302E_SOT23, Y1 8MHz

Commit message: [Development] Started porting the SMD version to the Proton C
Parts:
- removed C1, C2: 22p, Capacitor_SMD:C_0805_2012Metric_Pad1.15x1.40mm_HandSolder, symbol Device:C_Small
- removed U1: STM32F303CCT6, Package_QFP:LQFP-48_7x7mm_P0.5mm, symbol acheronSymbols:STM32F303CCT6
- removed Y1: 8MHz, acheronComponents:Crystal_SMD_5032-4Pin_5.0x3.2mm, symbol Device:Crystal_GND24
- added U?: proton_c, symbol proton_c:proton_c
Connections:
- net labels removed: XTAL1, XTAL2
- wire segments 648 -> 617
- no-connect marks 10 -> 11

Commit message: [Development] Started porting the SMD version to the Proton C
Parts:
- removed CSin1, CSout1, CVBus1, CVBus2, CVBus3: 100n, Capacitor_SMD:C_0805_2012Metric_Pad1.15x1.40mm_HandSolder, symbol Device:C_Small
- removed CVBus4: 1u, Capacitor_SMD:C_0402_1005Metric, symbol Device:C_Small
- removed CVBus5: 4.7u, Capacitor_SMD:C_0805_2012Metric_Pad1.15x1.40mm_HandSolder, symbol Device:C_Small
- removed DF1: RB060M-60TR, acheronComponents:D_SOD-123, symbol Device:D_Schottky_Small
- removed DS1: 1N4148, Diode_SMD:D_0805_2012Metric_Pad1.15x1.40mm_HandSolder, symbol Device:D
- removed F1: 1A, Fuse:Fuse_0805_2012Metric_Pad1.15x1.40mm_HandSolder, symbol Device:Polyfuse_Small
- removed U2: MCP1700-3302E_SOT23, Package_TO_SOT_SMD:SOT-23, symbol Regulator_Linear:MCP1700-3302E_SOT23
- U1: renamed from U?; value proton_c -> ProtonC
Connections:
- net 3.3V: now also RA2.2, RB2.2
- net 5V: now also U1.5V (VBUS(5V_RAW)); no longer RA2.2, RB2.2, U1.A3|5v (A3(5v_shifted)), U1.CHRG (CHRG(5v))
- net Col1: now also U1.B0 (PB0)
Other:
- note removed: "Polyfuse PPTC RTC"
- note removed: "Power supply and protection circuit"
- note removed: "Voltage regulation\ncapacitor bank\n"
